File: circuit/PaganiniClock.brd (EAGLE design)
At the start: 96.5 x 48.3 mm, 15 parts, among them IC1 4094, IC2 4094, M1 Digispark, M2 RTC-DS3231

Commit message: Add files via upload
Parts:
- moved S1 35.6 mm to (67.3, 41.9), turned to 180 degrees
- moved S2 35.6 mm to (67.3, 6.35), turned to 0 degrees
- moved R3 24.3 mm to (52.1, 8.89)
- moved R4 24.3 mm to (52.1, 39.4)
- moved C1 4.26 mm to (48.3, 39.4), turned to 270 degrees
- moved R2 4.07 mm to (52.1, 24.1), turned to 90 degrees
- moved C2 4.02 mm to (48.3, 8.89), turned to 90 degrees
- moved R1 2.62 mm to (48.3, 24.1), turned to 270 degrees
- moved IC1 0.63 mm to (34.3, 39.4)
Connections:
- net N$18: now also S2.3; no longer S1.4
- net N$20: now also S1.4; no longer S2.3
Routing:
- net BUTTONS: track 77.2 -> 48.5 mm
- net +5V: track 204.4 -> 218.9 mm
- net SCK: track 53.1 -> 60.5 mm
- net N$20: track 6.28 -> 12.4 mm
- net N$18: track 6.28 -> 12.4 mm
- net N$1: track 5.43 -> 9.99 mm
- net K: track 49.2 -> 52.1 mm
- net C: track 43.9 -> 46.8 mm
- net E: track 61.3 -> 59.0 mm
- net G1: track 60.0 -> 57.8 mm
- net J: track 46.7 -> 46.0 mm
- net A2: track 45.4 -> 44.8 mm
- net A1: track 37.1 -> 36.5 mm
- net H: track 32.1 -> 31.4 mm
- net SER-OUT: track 45.2 -> 44.6 mm
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